Commit message: Simulator steering now working.

File: otter_description/urdf/materials.xacro (robot description, xacro)
@@ -25,6 +25,12 @@
     <color rgba="1.0 1.0 1.0 1.0"/>
   </material>
-  <material name="dark_grey"><color rgba="0.2 0.2 0.2 1.0" /></material>
-  <material name="light_grey"><color rgba="0.4 0.4 0.4 1.0" /></material>
-  <material name="yellow"><color rgba="0.8 0.8 0.0 1.0" /></material>
+  <material name="dark_grey">
+    <color rgba="0.2 0.2 0.2 1.0" />
+  </material>
+  <material name="light_grey">
+    <color rgba="0.4 0.4 0.4 1.0" />
+  </material>
+  <material name="yellow">
+    <color rgba="0.8 0.8 0.0 1.0" />
+  </material>
 </robot>

File: otter_description/urdf/otter.xacro (robot description, xacro)
@@ -1,12 +1,11 @@
 <?xml version="1.0"?>
-<!-- Revolute-Revolute Manipulator -->
 <robot name="otter" xmlns:xacro="http://www.ros.org/wiki/xacro">
   <!-- Constants for robot dimensions -->
   <xacro:property name="PI" value="3.1415926535897931"/>
-  <xacro:property name="mass" value="16.523" /> <!-- arbitrary value for mass -->
-  <xacro:property name="width" value="0.31" /> <!-- Square dimensions (widthxwidth) of beams -->
+  <xacro:property name="mass" value="16.523" />
+  <xacro:property name="width" value="0.31" />
   <xacro:property name="length" value="0.42" />
-  <xacro:property name="height1" value="0.184" /> <!-- Link 1 -->
-  <xacro:property name="axel_offset" value="0.05" /> <!-- Space btw top of beam and the each joint -->
+  <xacro:property name="height1" value="0.184" />
+  <xacro:property name="axel_offset" value="0.05" />
   <xacro:property name="wheelbase" value="0.262" />
   <xacro:property name="track" value="0.37559" />
@@ -77,5 +76,5 @@
   <!-- Wheels -->
   <xacro:macro name="wheel" params="prefix *joint_pose">
-  <link name="${prefix}_wheel_link">
+    <link name="${prefix}_wheel_link">
       <visual>
         <origin xyz="0 0 0" rpy="${PI/2} 0 0"/>
@@ -103,5 +102,5 @@
       <material>Gazebo/DarkGrey</material>
     </gazebo>
-    <joint name="${prefix}_wheel" type="continuous">
+    <joint name="${prefix}_wheel_joint" type="continuous">
       <parent link="base_link"/>
       <child link="${prefix}_wheel_link" />
@@ -109,9 +108,7 @@
       <axis xyz="0 1 0" />
     </joint>
-    <!-- In reality, Jackal has only two motors, one per side. However, it's more
-         straightforward for Gazebo to simulate as if there's an actuator per wheel. -->
     <transmission name="${prefix}_wheel_trans">
       <type>transmission_interface/SimpleTransmission</type>
-      <joint name="${prefix}_wheel">
+      <joint name="${prefix}_wheel_joint">
         <hardwareInterface>hardware_interface/VelocityJointInterface</hardwareInterface>
       </joint>
@@ -132,4 +129,4 @@
   <xacro:wheel prefix="rear_right">
     <origin xyz="${-wheelbase/2} ${-track/2} ${wheel_vertical_offset}" rpy="0 0 0" />
-</xacro:wheel>
+  </xacro:wheel>
 </robot>
